File: KiCad/Elephant0.9.2/Elephant0.9.2.kicad_pcb (KiCad board)
At the start: 2 copper layers, 64.5 x 41.9 mm, 61 parts, among them J1 Conn_01x04_Pin, J2 Conn_01x05_Pin, SW1 SW_TILT, U1 LT8640, U3 SSM2518, U4 M95M04, U5 STM32F401CCUx, Y1 32.768kHz, 6pF, 50kΩ, Y2 16MHz, 7pF, 60Ω

Commit message: Added the audio system with a way to test it.
Parts:
- added ?: , , F.Cu at (74.4, 25.9)
- added JP1: SolderJumper_2_Open, Jumper:SolderJumper-2_P1.3mm_Open_Pad1.0x1.5mm, F.Cu at (36.6, 56.1)
- added REF**1: pinhole, paul:pinhole, F.Cu at (74.4, 27.9)
- C11, C12, C13, C15, C16, C18, C5, C6, C7, C8, C9: footprint Capacitor_SMD:C_0201_0603Metric -> Capacitor_SMD:C_0603_1608Metric
- J2: value Conn_01x05_Pin -> Conn_01x07_Pin; footprint Connector_JST:JST_PH_B5B-PH-K_1x05_P2.00mm_Vertical -> Connector_JST:JST_PH_B7B-PH-K_1x07_P2.00mm_Vertical
- moved R1 0.99 mm to (38.5, 53.8)
- moved J2 0.43 mm to (78.2, 39.0)
Connections:
- J2 pad 1: /jtms_swdio -> +3.3V
- J2 pad 2: /jtck_swclk -> /jtms_swdio
- J2 pad 3: /jtdi -> /jtck_swclk
- J2 pad 4: /jtdo-swo -> /jtdi
- J2 pad 5: /jtrst -> /jtdo-swo
Routing:
- net +9V: track 17.7 -> 25.1 mm
- net /pwr_buck: track 39.4 -> 45.1 mm
- net GND: track 118.8 -> 114.8 mm, vias 24 -> 25
- net /jtdo-swo: track 26.6 -> 28.0 mm
- net /osc32_in: track 13.1 -> 14.2 mm
- net /jtdi: track 19.5 -> 20.5 mm
- net /jtrst: track 29.3 -> 30.3 mm
- net Net-(SW1-A): track 9.64 -> 8.84 mm
- net Net-(C11-Pad1): track 11.9 -> 12.7 mm
- net Net-(C5-Pad1): track 11.6 -> 12.2 mm
- net +BATT: track 13.5 -> 14.1 mm
- net /jtms_swdio: track 16.9 -> 17.4 mm
- net /jtck_swclk: track 17.8 -> 18.3 mm
- removed copper zone on B.Cu, net (none)
- removed copper zone on F.Cu, net (none)
Other:
- outline, holes or cut-outs redrawn
